File: hardware/kicad/pa-telaio.kicad_sch (KiCad schematic)
At the start: 127 parts, among them J201 IN L (112AX), J202 IN R (112AX), J203 OUT L (112AX), J204 OUT R (112AX), J205 DC 9V (NEB/J 21C), J206 PEDALE (112BX), J207 MIDI IN (TRS tipo A), J208 MIDI OUT (TRS tipo A), J209 microSD, Q101 J201, Q102 J201, Q103 J201, Q104 J201, SW201 INST/LINE, SW202 PRE, SW203 true bypass, SW204 K1, SW205 K2, U1 TLC2272, U2 TLC2272, U301 H11L1M

Commit message: Schema KiCad disegnato: 10 pagine A3 con fili e un foglio per blocco, PDF; netlist verificata, ERC pulito, 6 mutazioni
Parts:
- removed A1: Daisy Seed3, symbol PA:SEED3
- removed A201: OLED 2,42 pollici I2C, symbol PA:OLED
- removed C1, C2: 100µF, Capacitor_THT:CP_Radial_D5.0mm_P2.50mm, symbol PA:CP
- removed C10, C12, C14, C15, C17, C7: 10µF, Capacitor_THT:CP_Radial_D5.0mm_P2.50mm, symbol PA:CP
- removed C101, C105: 47n, Capacitor_THT:C_Rect_L7.2mm_W3.5mm_P5.00mm_FKS2_FKP2_MKS2_MKP2, symbol PA:C
- removed C102, C106: 47u/16V, Capacitor_THT:CP_Radial_D5.0mm_P2.50mm, symbol PA:CP
- removed C103, C107: 220n, Capacitor_THT:C_Rect_L7.2mm_W3.5mm_P5.00mm_FKS2_FKP2_MKS2_MKP2, symbol PA:C
- removed C104, C108: 1u, Capacitor_THT:C_Rect_L7.2mm_W3.5mm_P5.00mm_FKS2_FKP2_MKS2_MKP2, symbol PA:C
- removed C109: 22u/16V, Capacitor_THT:CP_Radial_D5.0mm_P2.50mm, symbol PA:CP
- removed C11, C18, C3: 100nF, Capacitor_THT:C_Disc_D5.0mm_W2.5mm_P5.00mm, symbol PA:C
- removed C110: 100u/16V, Capacitor_THT:CP_Radial_D5.0mm_P2.50mm, symbol PA:CP
- removed C111: 100n, Capacitor_THT:C_Disc_D5.0mm_W2.5mm_P2.50mm, symbol PA:C
- removed C13, C16: 390pF, Capacitor_THT:C_Disc_D5.0mm_W2.5mm_P5.00mm, symbol PA:C
- removed C19, C20: 100pF, Capacitor_THT:C_Disc_D5.0mm_W2.5mm_P5.00mm, symbol PA:C
- removed C301, C302: 100n, symbol PA:C
- removed C4: 47µF, Capacitor_THT:CP_Radial_D5.0mm_P2.50mm, symbol PA:CP
- removed C5, C8: 100nF, Capacitor_THT:C_Rect_L7.2mm_W3.5mm_P5.00mm_FKS2_FKP2_MKS2_MKP2, symbol PA:C
- removed C6, C9: 2.2nF, Capacitor_THT:C_Disc_D5.0mm_W2.5mm_P5.00mm, symbol PA:C
- removed D1: 1N5817, Diode_THT:D_DO-41_SOD81_P10.16mm_Horizontal, symbol PA:D
- removed D201: LED bypass, symbol PA:LED
- removed D202: LED, symbol PA:LED
- removed D301: 1N4148, symbol PA:D
- removed ENC201: PEC11R, symbol PA:ENC
- removed H201: massa L0 (vite), symbol PA:MASSA
- removed H202: massa L1 (torretta), symbol PA:MASSA
- removed J201: IN L (112AX), symbol PA:JACK_TS
- removed J202: IN R (112AX), symbol PA:JACK_TS
- removed J203: OUT L (112AX), symbol PA:JACK_TS
- removed J204: OUT R (112AX), symbol PA:JACK_TS
- removed J205: DC 9V (NEB/J 21C), symbol PA:DC
- removed J206: PEDALE (112BX), symbol PA:JACK_TRS
- removed J207: MIDI IN (TRS tipo A), symbol PA:JACK_TRS
- removed J208: MIDI OUT (TRS tipo A), symbol PA:JACK_TRS
- removed J209: microSD, symbol PA:MICROSD
- removed Q101, Q102, Q103, Q104: J201, Package_TO_SOT_THT:TO-92_Inline, symbol PA:NJFET
- removed R1: 3R3, Resistor_THT:R_Axial_DIN0207_L6.3mm_D2.5mm_P7.62mm_Horizontal, symbol PA:R
- removed R10, R7: 1K, Resistor_THT:R_Axial_DIN0207_L6.3mm_D2.5mm_P7.62mm_Horizontal, symbol PA:R
- removed R101, R106, R110, R115, R5, R6, R8, R9: 1M, Resistor_THT:R_Axial_DIN0207_L6.3mm_D2.5mm_P7.62mm_Horizontal, symbol PA:R
- removed R102, R107, R111, R116: 1k, Resistor_THT:R_Axial_DIN0207_L6.3mm_D2.5mm_P7.62mm_Horizontal, symbol PA:R
- removed R103, R112: 27k, Resistor_THT:R_Axial_DIN0207_L6.3mm_D2.5mm_P7.62mm_Horizontal, symbol PA:R
- removed R104, R113: 22k, Resistor_THT:R_Axial_DIN0207_L6.3mm_D2.5mm_P7.62mm_Horizontal, symbol PA:R
- removed R105, R114: 220R, Resistor_THT:R_Axial_DIN0207_L6.3mm_D2.5mm_P7.62mm_Horizontal, symbol PA:R
- removed R108, R117: 20k, Resistor_THT:R_Axial_DIN0207_L6.3mm_D2.5mm_P7.62mm_Horizontal, symbol PA:R
- removed R109, R118: 15k, Resistor_THT:R_Axial_DIN0207_L6.3mm_D2.5mm_P7.62mm_Horizontal, symbol PA:R
- removed R11, R12, R15, R16, R3, R4: 10K, Resistor_THT:R_Axial_DIN0207_L6.3mm_D2.5mm_P7.62mm_Horizontal, symbol PA:R
- removed R119: 39k, Resistor_THT:R_Axial_DIN0207_L6.3mm_D2.5mm_P7.62mm_Horizontal, symbol PA:R
- removed R120: 10k, Resistor_THT:R_Axial_DIN0207_L6.3mm_D2.5mm_P7.62mm_Horizontal, symbol PA:R
- removed R13, R17: 100R, Resistor_THT:R_Axial_DIN0207_L6.3mm_D2.5mm_P7.62mm_Horizontal, symbol PA:R
- removed R14, R18: 100K, Resistor_THT:R_Axial_DIN0207_L6.3mm_D2.5mm_P7.62mm_Horizontal, symbol PA:R
- removed R2: 10R, Resistor_THT:R_Axial_DIN0207_L6.3mm_D2.5mm_P7.62mm_Horizontal, symbol PA:R
- removed R201: 10k (Rs L), symbol PA:R
- removed R202: 10k (Rs R), symbol PA:R
- removed R203: 3k3 (Rsh L), symbol PA:R
- removed R204: 3k3 (Rsh R), symbol PA:R
- removed R205: 47k (GAIN L), symbol PA:R
- removed R206: 47k (GAIN R), symbol PA:R
- removed R207: 4k7, symbol PA:R
- removed R208: 1k, symbol PA:R
- removed R301: 220, symbol PA:R
- removed R302: 270, symbol PA:R
- removed R303, R304: 10, symbol PA:R
- removed R305, R306, R307, R308, R309: 47k, symbol PA:R
- removed RV101, RV102: 100k, Potentiometer_THT:Potentiometer_Bourns_3296W_Vertical, symbol PA:TRIM
- removed RV201: GAIN C50K doppio, symbol PA:POT2
- removed RV202, RV203, RV204, RV205, RV206, RV207: B10K, symbol PA:POT
- removed SW201: INST/LINE, symbol PA:DPDT
- removed SW202: PRE, symbol PA:DPDT
- removed SW203: true bypass, symbol PA:3PDT
- removed SW204: K1, symbol PA:TASTO
- removed SW205: K2, symbol PA:TASTO
- removed U1, U2: TLC2272, Package_DIP:DIP-8_W7.62mm_Socket, symbol PA:TLC2272
- removed U301: H11L1M, symbol PA:H11L1
Connections:
- no-connect marks 21 -> 0
Other:
- added sheet Alimentazione (f01_alimentazione.kicad_sch)
- added sheet Buffer d'ingresso (f04_buffer_ingresso.kicad_sch)
- added sheet Buffer d'uscita (f05_buffer_uscita.kicad_sch)
- added sheet Controlli: pot, encoder, OLED, tasti, pedale (f08_controlli.kicad_sch)
- added sheet Daisy Seed3 (f07_seed.kicad_sch)
- added sheet Ingressi: jack, INST/LINE, PRE (f02_ingressi.kicad_sch)
- added sheet MIDI e microSD (f09_midi_sd.kicad_sch)
- added sheet Preamp JFET (schedina) (f03_preamp.kicad_sch)
- added sheet Uscite e true bypass (f06_uscite.kicad_sch)
- note added: "PA-TELAIO: schema elettrico"
- note added: "Strumento da tavolo su Daisy Seed3. Un foglio per blocco; fra un foglio e l'altro le reti passano per etichette globali con lo stesso nome."
- note added: "pagina 10"
- note added: "pagina 2"
- note added: "pagina 3"
- note added: "pagina 4"
- note added: "pagina 5"
- note added: "pagina 6"
- note added: "pagina 7"
- note added: "pagina 8"
- note added: "pagina 9"
- note removed: "Alimentazione, pedale, massa"
- note removed: "Controlli"
- note removed: "Ingressi e preamp"
- note removed: "Scheda MIDI"
- note removed: "Schedina preamp JFET"
- note removed: "Seed3 e operazionali"
- note removed: "Uscite e true bypass"
- note removed: "Veroboard: alimentazione, ingressi, uscite"
- note removed: "microSD"
- title: PA-TELAIO -> PA-TELAIO: indice dei fogli
